File: pcb/RH023.2/RH023.2.brd (EAGLE design)
At the start: 99.1 x 78.7 mm, 32 parts, among them CN1 USB, U2 FT232RLSSOP, U3 REG1117

Commit message: fixed unattached nets
Connections:
- net N$19: now also LED5.1
- net N$6: now also U4.P$5
Routing:
- net N$6: track 38.7 -> 79.8 mm, vias 0 -> 2
- net N$19: track 0.00 -> 34.7 mm, vias 0 -> 1
Changed lines of the file:
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@@
 <wire x1="77.3811" y1="51.0921" x2="77.42" y2="51.19" width="0.3048" layer="16"/>
 <wire x1="58.9788" y1="51.0921" x2="58.92" y2="51.19" width="0.3048" layer="16"/>
+<contactref element="U4" pad="P$5"/>
+<wire x1="61.0362" y1="24.1173" x2="58.9788" y2="24.1173" width="0.3048" layer="1"/>
+<wire x1="61.4934" y1="23.6601" x2="61.0362" y2="24.1173" width="0.3048" layer="1"/>
+<wire x1="62.1792" y1="22.9743" x2="61.4934" y2="23.6601" width="0.3048" layer="16"/>
+<wire x1="66.8655" y1="22.9743" x2="62.1792" y2="22.9743" width="0.3048" layer="16"/>
+<wire x1="75.6666" y1="31.7754" x2="66.8655" y2="22.9743" width="0.3048" layer="16"/>
+<wire x1="75.6666" y1="49.3776" x2="75.6666" y2="31.7754" width="0.3048" layer="1"/>
+<wire x1="77.3811" y1="51.0921" x2="75.6666" y2="49.3776" width="0.3048" layer="1"/>
+<wire x1="58.9788" y1="24.1173" x2="58.92" y2="24.175" width="0.3048" layer="1"/>
+<wire x1="77.3811" y1="51.0921" x2="77.42" y2="51.19" width="0.3048" layer="1"/>
+<via x="61.4934" y="23.6601" extent="1-16" drill="0.3048"/>
+<via x="75.6666" y="31.7754" extent="1-16" drill="0.3048"/>
 </signal>
 <signal name="N$7">
@@
 <signal name="N$19">
 <contactref element="U4" pad="P$17"/>
+<contactref element="LED5" pad="1"/>
+<wire x1="69.8373" y1="15.3162" x2="69.1515" y2="15.3162" width="0.3048" layer="1"/>
+<wire x1="74.9808" y1="20.4597" x2="69.8373" y2="15.3162" width="0.3048" layer="1"/>
+<wire x1="74.9808" y1="43.6626" x2="74.9808" y2="20.4597" width="0.3048" layer="1"/>
+<wire x1="77.3811" y1="46.0629" x2="74.9808" y2="43.6626" width="0.3048" layer="16"/>
+<wire x1="69.1515" y1="15.3162" x2="69.08" y2="15.285" width="0.3048" layer="1"/>
+<wire x1="77.3811" y1="46.0629" x2="77.42" y2="46.11" width="0.3048" layer="16"/>
+<via x="74.9808" y="43.6626" extent="1-16" drill="0.3048"/>
 </signal>
 <signal name="N$21">
